File: PCB/Smart_Door_Sensor/Smart_Door_Sensor.kicad_pcb (KiCad board)
At the start: 2 copper layers, 64.8 x 57.2 mm, 11 parts, among them SW1 SW_SPDT, SW2 SW_SPDT, U1 Wemos_Lolin32_Lite, U2 Door_Sensor

Commit message: V0.6.2 Finalised PCB V1.0
Other:
- board text added: "Sean Price"
- board text added: "Smart Door Sensor"
- board text added: "V1.0"
Changed lines of the file:
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@@
       (layerselection 0x00010fc_ffffffff)
       (disableapertmacros false)
-      (usegerberextensions false)
-      (usegerberattributes true)
-      (usegerberadvancedattributes true)
-      (creategerberjobfile true)
+      (usegerberextensions true)
+      (usegerberattributes false)
+      (usegerberadvancedattributes false)
+      (creategerberjobfile false)
       (svguseinch false)
       (svgprecision 6)
@@
       (plotinvisibletext false)
       (sketchpadsonfab false)
-      (subtractmaskfromsilk false)
+      (subtractmaskfromsilk true)
       (outputformat 1)
       (mirror false)
-      (drillshape 1)
+      (drillshape 0)
       (scaleselection 1)
-      (outputdirectory "")
+      (outputdirectory "../Smart_Door_Sensor_V1_Gerber/")
     )
   )
@@
   )
   (gr_rect (start 55.88 68.58) (end 120.65 125.73) (layer "Edge.Cuts") (width 0.1) (fill none))
+  (gr_text "Smart Door Sensor" (at 67.945 80.645) (layer "F.SilkS")
+    (effects (font (size 1.5 1.5) (thickness 0.3)))
+  )
+  (gr_text "Sean Price" (at 57.15 85.725) (layer "F.SilkS")
+    (effects (font (size 1.5 1.5) (thickness 0.3)) (justify left))
+  )
+  (gr_text "V1.0" (at 59.69 83.185) (layer "F.SilkS")
+    (effects (font (size 1.5 1.5) (thickness 0.3)))
+  )
   (segment (start 98.36 111.06) (end 97.79 110.49) (width 1.5) (layer "F.Cu") (net 1))
   (segment (start 98.36 113.03) (end 98.36 111.06) (width 1.5) (layer "F.Cu") (net 1))
